Commit message: remove visual contact points

File: examples/Atlas/urdf/atlas_minimal_contact_glued_foot.urdf (robot description, URDF)
Before this commit: robot atlas, 29 links, 28 joints
Links:
- link l_foot: geometry collision sphere radius=0; collision sphere radius=0
- link l_hand: geometry collision sphere radius=0; collision sphere radius=0
- link l_lleg: geometry collision sphere radius=0; visual mesh filename=meshes/l_lleg.wrl scale=1 1 1
- link l_uleg: geometry collision sphere radius=0; collision sphere radius=0
- link pelvis: geometry collision sphere radius=0; collision sphere radius=0
- link r_foot: geometry collision sphere radius=0; collision sphere radius=0
- link r_hand: geometry collision sphere radius=0; collision sphere radius=0
- link r_lleg: geometry collision sphere radius=0; visual mesh filename=meshes/r_lleg.wrl scale=1 1 1
- link r_uleg: geometry collision sphere radius=0; collision sphere radius=0
- link utorso: geometry collision sphere radius=0; collision sphere radius=0
